Commit message: update urdf

File: ros/src/cartographer_ros/cartographer_ros/urdf/backpack_2d.urdf (robot description, URDF)
Before this commit: robot cartographer_backpack_2d, 4 links, 3 joints
Links:
- removed link vertical_laser_link
- link base_link: geometry visual box size=0.6 0.3 0.25
Joints:
- removed joint vertical_laser_link_joint
- joint horizontal_laser_link_joint: origin xyz=0.1007 0 0.0558 -> xyz=0.0 0 0.0
