Commit message: change camera param

File: src/prius_description/urdf/prius.urdf (robot description, URDF)
Before this commit: robot prius, 24 links, 23 joints
Joints:
- joint left_camera_joint: origin xyz=1 -0.7 1.0 rpy=0 0.05 1.0 -> xyz=1 -0.7 1.0 rpy=0 0.05 0
- joint right_camera_joint: origin xyz=-1 -0.7 1.0 rpy=0 0.05 2.1416 -> xyz=-1 -0.7 1.0 rpy=0 0.05 3.14159

Commit message: add parking world

File: src/prius_description/urdf/prius.urdf (robot description, URDF)
Before this commit: robot prius, 24 links, 23 joints
Joints:
- joint back_camera_joint: origin xyz=0 1.45 1.4 rpy=0 0.05 1.5707 -> xyz=0 1.45 1.4 rpy=0 0 1.5707
- joint front_camera_joint: origin xyz=0 -0.4 1.4 rpy=0 0.05 -1.5707 -> xyz=0 -0.4 1.4 rpy=0 0 -1.5707
- joint left_camera_joint: origin xyz=1 -0.7 1.0 rpy=0 0.05 0 -> xyz=1 -0.7 1.0 rpy=0 0 0
- joint right_camera_joint: origin xyz=-1 -0.7 1.0 rpy=0 0.05 3.14159 -> xyz=-1 -0.7 1.0 rpy=0 0 3.14159

Commit message: add docs/prius.md

File: src/prius_description/urdf/prius.urdf (robot description, URDF)
Before this commit: robot prius, 24 links, 23 joints
Joints:
- joint back_camera_joint: origin xyz=0 1.45 1.4 rpy=0 0 1.5707 -> xyz=0 1.95 1.4 rpy=0 0 1.5707
- joint front_camera_joint: origin xyz=0 -0.4 1.4 rpy=0 0 -1.5707 -> xyz=0 -1.4 1.4 rpy=0 0 -1.5707
